Commit message: QHB：mapping framework

File: uav_simulator/gazebo_simulator/urdf/box.xacro (robot description, xacro)
@@ -1,4 +1,4 @@
 <?xml version="1.0"?>
-<robot xmlns:xacro="http://www.ros.org/wiki/xacro">
+<robot xmlns:xacro="http://www.ros.org/wiki/xacro" name="box_robot">
   <!-- Box Link -->
   <link name="base_link">
@@ -20,5 +20,13 @@
     </inertial>
   </link>
-  <xacro:include filename="$(find learning_gazebo)/urdf/camera_sensor.xacro"/>
+  <!-- 包含相机的 xacro 文件 -->  <!-- 相机相对于父链接（parent）的位姿 -->
+  <xacro:include filename="$(find gazebo_simulator)/urdf/camera_sensor.xacro"/>
   <xacro:camera_sensor parent="base_link" xyz="0 0 0.3" rpy="0 0 0"/>
+  <!-- 包含激光雷达的 xacro 文件 -->
+  <!-- <joint name="lidar_platform" type="fixed" >
+    <parent link="base_link" />
+    <child link="lidar_link" />
+    <origin xyz="0 0 0.5" rpy="0 0 0" />
+  </joint>
+  <xacro:include filename="$(find gazebo_simulator)/urdf/livox_mid360.xacro"/> -->
 </robot>

File: uav_simulator/gazebo_simulator/urdf/camera_sensor.xacro (robot description, xacro)
@@ -1,6 +1,7 @@
 <?xml version="1.0"?>
-<robot xmlns:xacro="http://www.ros.org/wiki/xacro">
+<robot xmlns:xacro="http://www.ros.org/wiki/xacro"  name="camera_sim">
   <!-- Camera Sensor -->
   <xacro:macro name="camera_sensor" params="parent xyz rpy">
+    <!-- 定义了一个相机的实体 -->
     <link name="camera_link">
       <visual>
@@ -17,15 +18,10 @@
       </inertial>
     </link>
-    <joint name="camera_joint" type="fixed">
-      <parent link="${parent}"/>
-      <child link="camera_link"/>
-      <origin xyz="${xyz}" rpy="${rpy}"/>
-    </joint>
-    <!-- Gazebo Camera Plugin -->
+    <!-- 使用Gazebo Camera Plugin，给相机实体添加仿真相机 -->
     <gazebo reference="camera_link">
-      <sensor type="camera" name="camera_sensor">
+      <sensor type="depth" name="camera_sensor">
         <update_rate>30.0</update_rate>
         <camera name="camera">
-          <horizontal_fov>1.047</horizontal_fov>
+          <horizontal_fov>1.39616</horizontal_fov>
           <image>
             <width>640</width>
@@ -35,5 +31,5 @@
           <clip>
             <near>0.1</near>
-            <far>100</far>
+            <far>20</far>
           </clip>
         </camera>
@@ -41,19 +37,25 @@
           <alwaysOn>true</alwaysOn>
           <updateRate>30.0</updateRate>
-          <cameraName>camera</cameraName>
-          <imageTopicName>color/image_raw2</imageTopicName>
-          <cameraInfoTopicName>color/camera_info2</cameraInfoTopicName>
-          <depthImageTopicName>depth/image_raw2</depthImageTopicName>
-          <depthCameraInfoTopicName>depth/camera_info2</depthCameraInfoTopicName>
-          <frameName>camera_link</frameName>
-          <hackBaseline>0.07</hackBaseline>
+          <cameraName>camera2</cameraName>
+          <imageTopicName>rgb/image_raw</imageTopicName>
+          <cameraInfoTopicName>rgb/camera_info</cameraInfoTopicName>
+          <depthImageTopicName>depth/image_raw</depthImageTopicName>
+          <depthCameraInfoTopicName>depth/camera_info</depthCameraInfoTopicName>
+          <frameName>support_depth</frameName>
+          <!-- <hackBaseline>0.07</hackBaseline>
           <distortionK1>0.0</distortionK1>
           <distortionK2>0.0</distortionK2>
           <distortionK3>0.0</distortionK3>
           <distortionT1>0.0</distortionT1>
-          <distortionT2>0.0</distortionT2>
+          <distortionT2>0.0</distortionT2> -->
         </plugin>
       </sensor>
     </gazebo>
+    <!-- 定义了一个固定的关节，用于连接camera_link和parent -->
+    <joint name="camera_joint" type="fixed">
+      <parent link="${parent}"/>
+      <child link="camera_link"/>
+      <origin xyz="${xyz}" rpy="${rpy}"/>
+    </joint>
   </xacro:macro>
 </robot>
