Commit message: 1

File: uav_simulator/jackal/jackal_description/urdf/jackal.urdf.xacro (robot description, xacro)
@@ -223,7 +223,7 @@
   </joint>
   <xacro:include filename="$(find jackal_description)/urdf/VLP_16.urdf.xacro"/>
-    <xacro:VLP_16 name="VLP_16" namespace="${namespace}/velodyne" parent="mid_mount" topic="velodyne_points" hz="100" samples="1800" gpu="true" max_range="11">
+    <xacro:VLP_16 name="VLP_16" namespace="${namespace}/velodyne" parent="mid_mount" topic="velodyne_points" hz="10" samples="1800" gpu="true" max_range="11">
 <!--  <xacro:VLP_16 name="VLP_16" namespace="${namespace}/velodyne" parent="mid_mount" topic="velodyne_points" hz="10" samples="440" gpu="false">-->
-    <origin xyz="0 0 0.134" rpy="0 0 0"/>
+    <origin xyz="0.2 0 0.134" rpy="0 ${0 * PI/18} 0"/>
 <!--    <origin xyz="0 0 0.135" rpy="0 0 0"/>-->
 <!--    <origin xyz="0 0 0.043" rpy="0 0 0"/>-->
